Commit message: Control barrier plugin gazebo

File: urdf/barrier.gazebo.xacro (robot description, xacro)
@@ -1,15 +1,3 @@
 <?xml version="1.0"?>
 <robot name="barrier_sim" xmlns:xacro="http://ros.org/wiki/xacro">
-  <gazebo reference="base_link">
-    <material>Gazebo/DarkGrey</material>
-  </gazebo>
-  <gazebo reference="motor">
-    <material>Gazebo/Black</material>
-  </gazebo>
-  <gazebo reference="gear">
-    <material>Gazebo/Grey</material>
-  </gazebo>
-  <gazebo reference="barrier">
-    <material>Gazebo/Yellow</material>
-  </gazebo>
 </robot>

File: urdf/barrier.urdf.xacro (robot description, xacro)
@@ -1,69 +1,65 @@
 <?xml version="1.0" ?>
 <robot name="barrier" xmlns:xacro="http://ros.org/wiki/xacro">
-  <xacro:include filename="$(find turtlebot3_description)/urdf/common_properties.xacro"/>
-  <xacro:include filename="$(find stage_arene_ros)/urdf/barrier.gazebo.xacro"/>
   <link name="world"/>
-  <joint name="base_joint" type="fixed">
+  <joint name="base_joint_1" type="fixed">
     <parent link="world"/>
-    <child link="base_link"/>
-    <origin xyz="0 0 0.001" rpy="0 0 0"/>
-  </joint>
-  <link name="base_link">
-    <visual>
-        <geometry>
-          <box size="0.05 0.05 0.005"/>
-        </geometry>
-        <material name="white"/>
-      </visual>
-    <collision>
-      <origin xyz="0 0 0.001" rpy="0 0 0"/>
-      <geometry>
-        <box size="0.05 0.05 0.005"/>
-      </geometry>
-    </collision>
-    <inertial>
-      <origin xyz="0 0 0" rpy="0 0 0"/>
-      <mass value="0.1"/>
-      <inertia ixx="0.0001" ixy="0" ixz="0"
-               iyy="0.0001" iyz="0"
-               izz="0.0001" />
-    </inertial>
-  </link>
-  <link name="motor">
-      <inertial>
-          <mass value="0.1"/>
-          <origin xyz="0 0 0"/>
-          <inertia ixx="0.01" ixy="0" ixz="0"
-                   iyy="0.01" iyz="0"
-                   izz="0.01" />
-      </inertial>
-      <collision>
-          <origin xyz="0 0 0" rpy="0 0 0"/>
-          <geometry>
-              <box size="0.04 0.037 0.02"/>
-          </geometry>
-      </collision>
-      <visual>
-            <geometry>
-                <box size="0.04 0.037 0.02"/>
-            </geometry>
-            <material name="black"/>
-        </visual>
-  </link>
-  <joint name="base_to_motor" type="fixed">
-      <parent link="base_link"/>
-      <child link="motor"/>
-      <origin xyz="0 0 0.0125"/>
-  </joint>
-  <link name="gear">
-    <inertial>
-      <mass value="0.1"/>
-      <origin xyz="0 0 0"/>
-      <inertia ixx="0.01" ixy="0" ixz="0"
-               iyy="0.01" iyz="0"
-               izz="0.01" />
-    </inertial>
-    <collision>
-      <origin xyz="0 0 0" rpy="0 0 0"/>
+    <child link="base_link_1"/>
+    <origin xyz="-1.5 0.9 0.01" rpy="0 0 1.57"/>
+  </joint>
+  <link name="base_link_1">
+    <visual>
+      <geometry>
+        <box size="0.05 0.05 0.005"/>
+      </geometry>
+    </visual>
+    <collision>
+      <origin xyz="0 0 0" rpy="0 0 0"/>
+      <geometry>
+        <box size="0.05 0.05 0.005"/>
+      </geometry>
+    </collision>
+    <inertial>
+      <origin xyz="0 0 0" rpy="0 0 0"/>
+      <mass value="0.1"/>
+      <inertia  ixx="0.0001" ixy="0" ixz="0"
+                iyy="0.0001" iyz="0"
+                izz="0.0001" />
+    </inertial>
+  </link>
+  <link name="motor_1">
+    <inertial>
+      <mass value="0.1"/>
+      <origin xyz="0 0 0" rpy="0 0 0"/>
+      <inertia  ixx="0.01" ixy="0" ixz="0"
+                iyy="0.01" iyz="0"
+                izz="0.01" />
+    </inertial>
+    <collision>
+      <origin xyz="0 0 0" rpy="0 0 0"/>
+      <geometry>
+        <box size="0.04 0.037 0.02"/>
+      </geometry>
+    </collision>
+    <visual>
+      <geometry>
+        <box size="0.04 0.037 0.02"/>
+      </geometry>
+    </visual>
+  </link>
+  <joint name="base_to_motor_1" type="fixed">
+    <parent link="base_link_1"/>
+    <child link="motor_1"/>
+    <origin xyz="0 0 0.0125" rpy="0 0 0"/>
+  </joint>
+  <link name="gear_1">
+    <inertial>
+      <mass value="0.1"/>
+      <origin xyz="0 0 0" rpy="0 0 0"/>
+      <inertia ixx="0.01" ixy="0" ixz="0"
+              iyy="0.01" iyz="0"
+              izz="0.01" />
+    </inertial>
+    <collision>
+      <origin xyz="0.01 0.021 0" rpy="-1.57 3.14 0"/>
       <geometry>
         <cylinder radius="0.01" length="0.005"/>
@@ -74,41 +70,195 @@
             <cylinder radius="0.01" length="0.005"/>
         </geometry>
-        <material name="gray"/>
-    </visual>
-  </link>
-  <joint name="motor_to_gear" type="fixed">
-      <parent link="motor"/>
-      <child link="gear"/>
-      <origin xyz="0.01 0.021 0.0" rpy="-1.57 3.14 0"/>
-  </joint>
-  <link name="barrier">
+    </visual>
+  </link>
+  <joint name="motor_to_gear_1" type="fixed">
+      <parent link="motor_1"/>
+      <child link="gear_1"/>
+      <origin xyz="0.01 0.021 0" rpy="-1.57 3.14 0"/>
+  </joint>
+  <link name="barrier_1">
     <inertial>
       <mass value="0.01"/>
-      <origin xyz="0 0 0"/>
-      <inertia ixx="0.01" ixy="0" ixz="0"
-               iyy="0.01" iyz="0"
-               izz="0.01" />
-    </inertial>
-    <collision>
-      <origin xyz="0.09 0.02 0.0005" rpy="0 0 0"/>
-      <geometry>
-        <box size="0.2 0.06 0.001"/>
-      </geometry>
-    </collision>
-    <visual>
-      <origin xyz="0.09 0.02 0.0005" rpy="0 0 0"/>
-      <geometry>
-        <box size="0.2 0.06 0.001"/>
-      </geometry>
-      <material name="dark"/>
-    </visual>
-  </link>
-  <joint name="gear_to_$(arg model_name)" type="revolute">
+      <origin xyz="0 0 0" rpy="0 0 0"/>
+      <inertia ixx="0.01" ixy="0" ixz="0"
+              iyy="0.01" iyz="0"
+              izz="0.01" />
+    </inertial>
+    <collision>
+      <origin xyz="0.09 0.02 0.0005" rpy="0 0 0"/>
+      <geometry>
+        <box size="0.2 0.06 0.001"/>
+      </geometry>
+    </collision>
+    <visual>
+      <origin xyz="0.09 0.02 0.0005" rpy="0 0 0"/>
+      <geometry>
+        <box size="0.2 0.06 0.001"/>
+      </geometry>
+    </visual>
+  </link>
+  <joint name="gear_to_barrier_1" type="revolute">
       <limit upper="1.57" lower="0" velocity="100" effort="100"/>
-      <origin xyz="0 0 0.0025"/>
+      <origin xyz="0 0 0.0025 " rpy="0 0 0"/>
       <axis xyz="0 0 1"/>
-      <parent link="gear"/>
-      <child link="barrier"/>
+      <parent link="gear_1"/>
+      <child link="barrier_1"/>
       <dynamics damping="0.1" friction="0.1"/>
   </joint>
+  <gazebo>
+    <plugin name="gazebo_ros_control" filename="libgazebo_ros_control.so">
+      <robotNamespace>/barrier_1</robotNamespace>
+    </plugin>
+  </gazebo>
+  <transmission name="gear_to_barrier_1_trans">
+    <type>transmission_interface/SimpleTransmission</type>
+    <actuator name="motor1">
+      <mechanicalReduction>1</mechanicalReduction>
+    </actuator>
+    <joint name="gear_to_barrier_1">
+      <hardwareInterface>hardware_interface/EffortJointInterface</hardwareInterface>
+    </joint>
+  </transmission>
+  <gazebo reference="base_link_1">
+    <material>Gazebo/DarkGrey</material>
+  </gazebo>
+  <gazebo reference="motor_1">
+    <material>Gazebo/Black</material>
+  </gazebo>
+  <gazebo reference="gear_1">
+    <material>Gazebo/Grey</material>
+  </gazebo>
+  <gazebo reference="barrier_1">
+    <material>Gazebo/Yellow</material>
+  </gazebo>
+  <joint name="base_joint_2" type="fixed">
+    <parent link="world"/>
+    <child link="base_link_2"/>
+    <origin xyz="-1.5 0.9 0.01" rpy="0 0 1.57"/>
+  </joint>
+  <link name="base_link_2">
+    <visual>
+      <geometry>
+        <box size="0.05 0.05 0.005"/>
+      </geometry>
+    </visual>
+    <collision>
+      <origin xyz="0 0 0" rpy="0 0 0"/>
+      <geometry>
+        <box size="0.05 0.05 0.005"/>
+      </geometry>
+    </collision>
+    <inertial>
+      <origin xyz="0 0 0" rpy="0 0 0"/>
+      <mass value="0.1"/>
+      <inertia  ixx="0.0001" ixy="0" ixz="0"
+                iyy="0.0001" iyz="0"
+                izz="0.0001" />
+    </inertial>
+  </link>
+  <link name="motor_2">
+    <inertial>
+      <mass value="0.1"/>
+      <origin xyz="0 0 0" rpy="0 0 0"/>
+      <inertia  ixx="0.01" ixy="0" ixz="0"
+                iyy="0.01" iyz="0"
+                izz="0.01" />
+    </inertial>
+    <collision>
+      <origin xyz="0 0 0" rpy="0 0 0"/>
+      <geometry>
+        <box size="0.04 0.037 0.02"/>
+      </geometry>
+    </collision>
+    <visual>
+      <geometry>
+        <box size="0.04 0.037 0.02"/>
+      </geometry>
+    </visual>
+  </link>
+  <joint name="base_to_motor_2" type="fixed">
+    <parent link="base_link_2"/>
+    <child link="motor_2"/>
+    <origin xyz="0 0 0.0125" rpy="0 0 0"/>
+  </joint>
+  <link name="gear_2">
+    <inertial>
+      <mass value="0.1"/>
+      <origin xyz="0 0 0" rpy="0 0 0"/>
+      <inertia ixx="0.01" ixy="0" ixz="0"
+              iyy="0.01" iyz="0"
+              izz="0.01" />
+    </inertial>
+    <collision>
+      <origin xyz="0.01 0.021 0" rpy="-1.57 3.14 0"/>
+      <geometry>
+        <cylinder radius="0.01" length="0.005"/>
+      </geometry>
+    </collision>
+    <visual>
+        <geometry>
+            <cylinder radius="0.01" length="0.005"/>
+        </geometry>
+    </visual>
+  </link>
+  <joint name="motor_to_gear_2" type="fixed">
+      <parent link="motor_2"/>
+      <child link="gear_2"/>
+      <origin xyz="0.01 0.021 0" rpy="-1.57 3.14 0"/>
+  </joint>
+  <link name="barrier_2">
+    <inertial>
+      <mass value="0.01"/>
+      <origin xyz="0 0 0" rpy="0 0 0"/>
+      <inertia ixx="0.01" ixy="0" ixz="0"
+              iyy="0.01" iyz="0"
+              izz="0.01" />
+    </inertial>
+    <collision>
+      <origin xyz="0.09 0.02 0.0005" rpy="0 0 0"/>
+      <geometry>
+        <box size="0.2 0.06 0.001"/>
+      </geometry>
+    </collision>
+    <visual>
+      <origin xyz="0.09 0.02 0.0005" rpy="0 0 0"/>
+      <geometry>
+        <box size="0.2 0.06 0.001"/>
+      </geometry>
+    </visual>
+  </link>
+  <joint name="gear_to_barrier_2" type="revolute">
+      <limit upper="1.57" lower="0" velocity="100" effort="100"/>
+      <origin xyz="0 0 0.0025 " rpy="0 0 0"/>
+      <axis xyz="0 0 1"/>
+      <parent link="gear_2"/>
+      <child link="barrier_2"/>
+      <dynamics damping="0.1" friction="0.1"/>
+  </joint>
+  <gazebo>
+    <plugin name="gazebo_ros_control" filename="libgazebo_ros_control.so">
+      <robotNamespace>/barrier_2</robotNamespace>
+    </plugin>
+  </gazebo>
+  <transmission name="gear_to_barrier_2_trans">
+    <type>transmission_interface/SimpleTransmission</type>
+    <actuator name="motor1">
+      <mechanicalReduction>1</mechanicalReduction>
+    </actuator>
+    <joint name="gear_to_barrier_2">
+      <hardwareInterface>hardware_interface/EffortJointInterface</hardwareInterface>
+    </joint>
+  </transmission>
+  <gazebo reference="base_link_2">
+    <material>Gazebo/DarkGrey</material>
+  </gazebo>
+  <gazebo reference="motor_2">
+    <material>Gazebo/Black</material>
+  </gazebo>
+  <gazebo reference="gear_2">
+    <material>Gazebo/Grey</material>
+  </gazebo>
+  <gazebo reference="barrier_2">
+    <material>Gazebo/Yellow</material>
+  </gazebo>
 </robot>
