Commit message: Simulation finie

File: urdf/barrier.urdf (robot description, URDF)
Before this commit: robot barrier, 17 links, 16 joints
Joints:
- joint base_joint_1_tl: origin xyz=-1.6 0.8 0.0001 rpy=0 0 1.57 -> xyz=-1.585 0.75 0.0001 rpy=0 0 1.57
- joint base_joint_2: origin xyz=-1.1 -1.6 0.01 rpy=0 0 3.14 -> xyz=-0.75 -1.65 0.01 rpy=0 0 0
- joint base_joint_2_tl: origin xyz=-1 -1.7 0.0001 rpy=0 0 0 -> xyz=-0.9 -1.7 0.0001 rpy=0 0 0

Commit message: avancées sur la simu et premiers tests sur l'arene

File: urdf/barrier.urdf (robot description, URDF)
Before this commit: robot barrier, 17 links, 16 joints
Links:
- link base_link_1_tl: geometry visual box size=0.1 0.03 0.005
- link base_link_2_tl: geometry visual box size=0.1 0.03 0.005

Commit message: Avec les tests que j'ai fait tout fonctionne

File: urdf/barrier.urdf (robot description, URDF)
Before this commit: robot barrier, 17 links, 16 joints
Links:
- removed link barrier_1
- removed link barrier_2
- removed link base_link_1
- removed link base_link_1_tl
- removed link base_link_2
- removed link base_link_2_tl
- removed link gear_1
- removed link gear_2
- removed link light_green_1
- removed link light_green_2
- removed link light_red_1
- removed link light_red_2
- removed link light_yellow_1
- removed link light_yellow_2
- removed link motor_1
- removed link motor_2
- added link barrier, mass 0.1; collision box size=0.3 0.08 0.005; visual box size=0.3 0.08 0.005
- added link base_link, mass 0.1; collision box size=0.05 0.05 0.005; visual box size=0.05 0.05 0.05
Joints:
- removed joint base_joint_1
- removed joint base_joint_1_tl
- removed joint base_joint_2
- removed joint base_joint_2_tl
- removed joint base_to_light_green_1
- removed joint base_to_light_green_2
- removed joint base_to_light_red_1
- removed joint base_to_light_red_2
- removed joint base_to_light_yellow_1
- removed joint base_to_light_yellow_2
- removed joint base_to_motor_1
- removed joint base_to_motor_2
- removed joint gear_to_barrier_1
- removed joint gear_to_barrier_2
- removed joint motor_to_gear_1
- removed joint motor_to_gear_2
- added joint barrier_joint: type fixed, parent world, child base_link, origin xyz=-1.50 0.9 0.025 rpy=0 0 1.57
- added joint base_to_barrier: type revolute, parent base_link, child barrier, origin xyz=-0.025 0.025 0.0 rpy=1.57 0 0, axis 0 0 1, limit lower=-1.57 upper=0 effort=1000 velocity=1.0
